File: mosfet-module.kicad_pcb (KiCad board)
At the start: 2 copper layers, 12 x 44 mm, 17 parts, among them J1 Terminal, J2 Conn_01x02_Socket, J3 Conn_01x02_Socket, M3 MountingHole_3.2mm_M3_Pad_Via, Q1 CSD17578Q5A, Q2 CSD17578Q5A

Commit message: update main PCB
Parts:
- moved M3 1.86 mm to (91.2, 108.8)
- moved M3 0.17 mm to (91.2, 70.8)
Other:
- board size 12 x 44 mm -> 12 x 48 mm
Changed lines of the file:
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@@
   )
   (footprint "MountingHole:MountingHole_3.2mm_M3_Pad_Via" (layer "F.Cu")
-    (at 91.313 106.947)
+    (at 91.15 108.802)
     (descr "Mounting Hole 3.2mm, M3")
     (tags "mounting hole 3.2mm m3")
@@
   )
   (footprint "MountingHole:MountingHole_3.2mm_M3_Pad_Via" (layer "F.Cu")
-    (at 91.313 70.752)
+    (at 91.15 70.802)
     (descr "Mounting Hole 3.2mm, M3")
     (tags "mounting hole 3.2mm m3")
@@
     )
   )
-  (gr_rect (start 85.155 66.802) (end 97.155 110.802)
+  (gr_rect (start 85.155 65.802) (end 97.155 113.802)
     (stroke (width 0.1) (type default)) (fill none) (layer "Edge.Cuts"))
   (gr_text "+" (at 85.471 103.759) (layer "F.SilkS")
@@
     (effects (font (size 1 1) (thickness 0.15)) (justify left bottom))
   )
-  (dimension (type aligned) (layer "B.Cu")
-    (pts (xy 85.155 66.802) (xy 85.155 110.802))
-    (height 8.955)
-    (gr_text "44.0000 mm" (at 74.4 88.802 90) (layer "B.Cu")
+  (dimension (type aligned) (layer "F.Cu")
+    (pts (xy 85.155 64.802) (xy 85.155 114.802))
+    (height 13.781)
+    (gr_text "50.0000 mm" (at 69.574 89.802 90) (layer "F.Cu")
       (effects (font (size 1.5 1.5) (thickness 0.3)))
     )
@@
   (segment (start 88.9 98.786) (end 89.682 99.568) (width 1.15) (layer "F.Cu") (net 7))
   (zone (net 4) (net_name "GND") (layer "F.Cu") (hatch edge 0.5)
-    (connect_pads (clearance 0.5))
+    (connect_pads yes (clearance 0.5))
     (min_thickness 0.25) (filled_areas_thickness no)
     (fill yes (thermal_gap 0.5) (thermal_bridge_width 0.5))
     (polygon
       (pts
-        (xy 84.836 111.379)
-        (xy 97.409 111.379)
+        (xy 84.836 114.935)
+        (xy 97.409 114.935)
         (xy 97.409 92.075)
         (xy 84.836 92.075)
@@
   (zone (net 4) (net_name "GND") (layer "F.Cu") (hatch edge 0.5)
     (priority 2)
-    (connect_pads (clearance 0.5))
+    (connect_pads yes (clearance 0.5))
     (min_thickness 0.25) (filled_areas_thickness no)
     (fill yes (thermal_gap 0.5) (thermal_bridge_width 0.5))
@@
         (xy 97.282 74.422)
         (xy 85.217 74.422)
-        (xy 85.217 66.802)
-        (xy 97.155 66.802)
+        (xy 85.217 64.897)
+        (xy 97.12325 64.897)
       )
     )

Commit message: update main PCB project files
Connections:
- M3 pad 1: (no net) -> GND
Routing:
- net Net-(J1-Pin_1): track 25.8 -> 23.8 mm
Changed lines of the file:
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@@
     (pad "1" thru_hole circle (at -1.697056 1.697056) (size 0.8 0.8) (drill 0.5) (layers "*.Cu" "*.Mask"))
     (pad "1" thru_hole circle (at 0 -2.4) (size 0.8 0.8) (drill 0.5) (layers "*.Cu" "*.Mask"))
-    (pad "1" thru_hole circle (at 0 0) (size 6.4 6.4) (drill 3.2) (layers "*.Cu" "*.Mask"))
+    (pad "1" thru_hole circle (at 0 0) (size 6.4 6.4) (drill 3.2) (layers "*.Cu" "*.Mask")
+      (net 4 "GND"))
     (pad "1" thru_hole circle (at 0 2.4) (size 0.8 0.8) (drill 0.5) (layers "*.Cu" "*.Mask"))
     (pad "1" thru_hole circle (at 1.697056 -1.697056) (size 0.8 0.8) (drill 0.5) (layers "*.Cu" "*.Mask"))
@@
     (effects (font (size 1 1) (thickness 0.15)) (justify left bottom))
   )
-  (dimension (type aligned) (layer "F.Cu")
-    (pts (xy 85.155 64.802) (xy 85.155 114.802))
-    (height 13.781)
-    (gr_text "50.0000 mm" (at 69.574 89.802 90) (layer "F.Cu")
-      (effects (font (size 1.5 1.5) (thickness 0.3)))
-    )
-    (format (prefix "") (suffix "") (units 3) (units_format 1) (precision 4))
-    (style (thickness 0.2) (arrow_length 1.27) (text_position_mode 0) (extension_height 0.58642) (extension_offset 0.5) keep_text_aligned)
-  )
   (dimension (type aligned) (layer "B.Cu")
     (pts (xy 85.155 66.802) (xy 97.155 66.802))
@@
   (segment (start 94.107 88.392) (end 94.234 87.503) (width 1.15) (layer "F.Cu") (net 3))
   (segment (start 94.234 89.408) (end 94.107 88.392) (width 1.15) (layer "F.Cu") (net 3))
-  (segment (start 94.234 87.503) (end 94.5 78) (width 1.15) (layer "F.Cu") (net 3))
+  (segment (start 94.234 87.503) (end 94.234 80) (width 1.15) (layer "F.Cu") (net 3))
   (via (at 93.175666 90.395777) (size 0.8) (drill 0.2) (layers "F.Cu" "B.Cu") (net 3))
   (via (at 93.175666 88.420223) (size 0.8) (drill 0.2) (layers "F.Cu" "B.Cu") (net 3))
